Commit message: until moveit config

File: src/manipulator_description/urdf/manipulator.urdf.xacro (robot description, xacro)
@@ -1,4 +1,10 @@
 <?xml version="1.0"?>
-<robot xmlns:xacro="http://www.ros.org/wiki/xacro" name="arduinobot">
+<robot xmlns:xacro="http://www.ros.org/wiki/xacro" name="manipulator">
+    <xacro:arg name="is_ignition" default="true"/>   <!-- Ignition simulation flag is used to enable/disable ignition features -->
+    <!-- Often you need to include different plugin tags, different frames, or different element names depending on whether you run
+     the model in Ignition (which changed some plugin names & SDF behavior) or in classic Gazebo. The is_ignition arg lets you
+     switch between those variants without maintaining two separate files.-->
+    <xacro:include filename="$(find manipulator_description)/urdf/manipulator_gazebo.xacro"/>
+    <xacro:include filename="$(find manipulator_description)/urdf/manipulator_ros2_control.xacro"/>
     <!-- Useful XACRO Variables (Properties) -->
     <xacro:property name="PI" value="3.14159265359" />
@@ -15,4 +21,26 @@
         </inertial>
     </xacro:macro>
+    <!-- Shared materials (RGBA, values 0..1) -->
+    <material name="mat_base">
+        <color rgba="0.0 0.2 0.8 1.0"/>   <!-- blue -->
+    </material>
+    <material name="mat_plate">
+        <color rgba="0.8 0.1 0.1 1.0"/>   <!-- red -->
+    </material>
+    <material name="mat_arm1">
+        <color rgba="0.1 0.8 0.2 1.0"/>   <!-- green -->
+    </material>
+    <material name="mat_arm2">
+        <color rgba="0.95 0.6 0.15 1.0"/> <!-- orange -->
+    </material>
+    <material name="mat_claw">
+        <color rgba="0.6 0.2 0.8 1.0"/>   <!-- purple -->
+    </material>
+    <material name="mat_gripper">
+        <color rgba="0.95 0.92 0.15 1.0"/><!-- yellow -->
+    </material>
+    <material name="mat_mesh_grey">
+        <color rgba="0.5 0.5 0.5 1.0"/>   <!-- fallback grey -->
+    </material>
     <!-- Links -->
     <link name="world"/>
@@ -24,4 +52,5 @@
                 <mesh filename="package://manipulator_description/meshes/basement.STL" scale="0.01 0.01 0.01"/>
             </geometry>
+            <material name="mat_base"/>
         </visual>
         <collision>
@@ -44,4 +73,5 @@
                 <mesh filename="package://manipulator_description/meshes/base_plate.STL" scale="0.01 0.01 0.01"/>
             </geometry>
+            <material name="mat_plate"/>
         </visual>
         <collision>
@@ -67,4 +97,5 @@
                 <mesh filename="package://manipulator_description/meshes/forward_drive_arm.STL" scale="0.01 0.01 0.01"/>
             </geometry>
+            <material name="mat_arm1"/>
         </visual>
         <collision>
@@ -90,4 +121,5 @@
                 <mesh filename="package://manipulator_description/meshes/horizontal_arm.STL" scale="0.01 0.01 0.01"/>
             </geometry>
+            <material name="mat_arm2"/>
         </visual>
         <collision>
@@ -113,4 +145,5 @@
                 <mesh filename="package://manipulator_description/meshes/claw_support.STL" scale="0.01 0.01 0.01"/>
             </geometry>
+            <material name="mat_claw"/>
         </visual>
         <collision>
@@ -133,4 +166,5 @@
                 <mesh filename="package://manipulator_description/meshes/right_finger.STL" scale="0.01 0.01 0.01"/>
             </geometry>
+            <material name="mat_gripper"/>
         </visual>
         <collision>
@@ -148,4 +182,5 @@
         <limit lower="-${PI / 2}" upper="0.0"
                effort="${effort}" velocity="${velocity}"/>
+        <dynamics damping="0.001" friction="0.001"/>
     </joint>
     <link name="gripper_left">
@@ -156,4 +191,5 @@
                 <mesh filename="package://manipulator_description/meshes/left_finger.STL" scale="0.01 0.01 0.01"/>
             </geometry>
+            <material name="mat_gripper"/>
         </visual>
         <collision>
@@ -171,4 +207,5 @@
         <limit lower="0.0" upper="${PI / 2}"
                effort="${effort}" velocity="${velocity}"/>
+        <dynamics damping="0.001" friction="0.001"/>
         <mimic joint="joint_4" multiplier="-1"/>   <!-- This joint mimics joint_4 means it will move in the opposite direction to joint_4 -->
     </joint>
